Commit message: before edit

File: src/excavator/excavator_description/urdf/excavator_with_kinect_gazebo.xacro (robot description, xacro)
@@ -3,6 +3,6 @@
     <xacro:include filename="$(find excavator_description)/urdf/excavator.xacro" />
     <xacro:include filename="$(find excavator_description)/urdf/sensors/kinect_gazebo.xacro" />
-    <xacro:property name="kinect_offset_x" value="-0.05" />
-    <xacro:property name="kinect_offset_y" value="0" />
+    <xacro:property name="kinect_offset_x" value="-0.1" />
+    <xacro:property name="kinect_offset_y" value="0.1" />
     <xacro:property name="kinect_offset_z" value="0.12" />
     <!-- kinect -->
