Commit message: successfully pass the excavator_description test

File: src/excavator/excavator_description/urdf/excavator.xacro (robot description, xacro)
@@ -22,7 +22,7 @@
     <!-- Macros -->
     <!-- Macro for Transmission -->
-    <xacro:macro name="transmission" params="joint_name">
+    <xacro:macro name="add_trans" params="joint_name">
         <!-- Transmission is important to link the joints and the controller -->
-        <xacro:transmission name="${joint_name}_trans">
+        <transmission name="${joint_name}_trans">
             <type>transmission_interface/SimpleTransmission</type>
             <joint name="${joint_name}" >
@@ -33,5 +33,5 @@
                 <mechanicalReduction>1</mechanicalReduction>
             </actuator>
-        </xacro:transmission>
+        </transmission>
     </xacro:macro>
     <!-- Excavator Model Macro -->
@@ -67,12 +67,12 @@
         </gazebo>
         <!-- Transmissions -->
-        <xacro:transmission joint_name="wheel1_joint"/>
-        <xacro:transmission joint_name="wheel4_joint"/>
-        <xacro:transmission joint_name="wheel2_joint"/>
-        <xacro:transmission joint_name="wheel3_joint"/>
-        <!-- <xacro:transmission joint_name="table_joint"/>
-        <xacro:transmission joint_name="link1_joint"/>
-        <xacro:transmission joint_name="link2_joint"/>
-        <xacro:transmission joint_name="ram_joint"/> -->
+        <xacro:add_trans joint_name="wheel1_joint"/>
+        <xacro:add_trans joint_name="wheel4_joint"/>
+        <xacro:add_trans joint_name="wheel2_joint"/>
+        <xacro:add_trans joint_name="wheel3_joint"/>
+        <!-- <xacro:add_trans joint_name="table_joint"/>
+        <xacro:add_trans joint_name="link1_joint"/>
+        <xacro:add_trans joint_name="link2_joint"/>
+        <xacro:add_trans joint_name="ram_joint"/> -->
         <!-- Gazebo Plugins -->
         <gazebo>

File: src/excavator/excavator_description/urdf/excavator_gazebo.xacro (robot description, xacro)
@@ -4,5 +4,5 @@
     <!-- 调用宏函数 -->
     <xacro:excavator/>
-    <xacro:transmission name="trans_table_joint">
+    <transmission name="trans_table_joint">
         <type>transmission_interface/SimpleTransmission</type>
         <joint name="table_joint">
@@ -13,6 +13,6 @@
             <mechanicalReduction>1</mechanicalReduction>
         </actuator>
-    </xacro:transmission>
-    <xacro:transmission name="trans_link1_joint">
+    </transmission>
+    <transmission name="trans_link1_joint">
         <type>transmission_interface/SimpleTransmission</type>
         <joint name="link1_joint">
@@ -23,6 +23,6 @@
             <mechanicalReduction>1</mechanicalReduction>
         </actuator>
-    </xacro:transmission>
-    <xacro:transmission name="trans_link2_joint">
+    </transmission>
+    <transmission name="trans_link2_joint">
         <type>transmission_interface/SimpleTransmission</type>
         <joint name="link2_joint">
@@ -33,6 +33,6 @@
             <mechanicalReduction>1</mechanicalReduction>
         </actuator>
-    </xacro:transmission>
-    <xacro:transmission name="trans_ram_joint">
+    </transmission>
+    <transmission name="trans_ram_joint">
         <type>transmission_interface/SimpleTransmission</type>
         <joint name="ram_joint">
@@ -43,5 +43,5 @@
             <mechanicalReduction>1</mechanicalReduction>
         </actuator>
-    </xacro:transmission>
+    </transmission>
     <gazebo>
         <plugin name="gazebo_ros_control" filename="libgazebo_ros_control.so">

Commit message: Fix the xacro parsing problem

File: src/excavator/excavator_description/urdf/excavator.xacro (robot description, xacro)
@@ -3,5 +3,6 @@
      Commit Version: 1.6.0-1-g15f4949  Build Version: 1.6.7594.29634
      For more information, please see http://wiki.ros.org/sw_urdf_exporter -->
-<robot name="excavator" xmlns:xacro="http://www.ros.org/wiki/xacro">
+<robot name="excavator"
+    xmlns:xacro="http://www.ros.org/wiki/xacro">
     <!-- PROPERTY LIST -->
     <xacro:property name="M_PI" value="3.1415926"/>
@@ -26,5 +27,5 @@
         <transmission name="${joint_name}_trans">
             <type>transmission_interface/SimpleTransmission</type>
-            <joint name="${joint_name}" >
+            <joint name="${joint_name}">
                 <hardwareInterface>hardware_interface/VelocityJointInterface</hardwareInterface>
             </joint>
@@ -77,6 +78,5 @@
         <!-- Gazebo Plugins -->
         <gazebo>
-            <plugin name="differential_drive_controller_front"
-                    filename="libgazebo_ros_diff_drive.so">
+            <plugin name="differential_drive_controller_front" filename="libgazebo_ros_diff_drive.so">
                 <rosDebugLevel>Debug</rosDebugLevel>
                 <publishWheelTF>true</publishWheelTF>
@@ -99,6 +99,5 @@
                 <robotBaseFrame>base_footprint</robotBaseFrame>
             </plugin>
-            <plugin name="differential_drive_controller_back"
-                    filename="libgazebo_ros_diff_drive.so">
+            <plugin name="differential_drive_controller_back" filename="libgazebo_ros_diff_drive.so">
                 <rosDebugLevel>Debug</rosDebugLevel>
                 <publishWheelTF>true</publishWheelTF>
@@ -144,38 +143,21 @@
         <link name="chassis">
             <inertial>
-                <origin
-                xyz="0.0044428 -5.5511E-17 -0.010796"
-                rpy="0 0 0" />
-                <mass
-                value="10.503" />
-                <inertia
-                ixx="0.029632"
-                ixy="1.9665E-18"
-                ixz="-9.9529E-05"
-                iyy="0.059252"
-                iyz="1.8828E-16"
-                izz="0.086263" />
-            </inertial>
-            <visual>
-                <origin
-                xyz="0 0 0"
-                rpy="0 0 0" />
-                <geometry>
-                <mesh
-                    filename="package://excavator_description/meshes/chassis.STL" />
-                </geometry>
-                <material
-                name="">
-                <color
-                    rgba="0.52941 0.54902 0.54902 1" />
-                </material>
-            </visual>
-            <collision>
-                <origin
-                xyz="0 0 0"
-                rpy="0 0 0" />
-                <geometry>
-                <mesh
-                    filename="package://excavator_description/meshes/chassis.STL" />
+                <origin xyz="0.0044428 -5.5511E-17 -0.010796" rpy="0 0 0" />
+                <mass value="10.503" />
+                <inertia ixx="0.029632" ixy="1.9665E-18" ixz="-9.9529E-05" iyy="0.059252" iyz="1.8828E-16" izz="0.086263" />
+            </inertial>
+            <visual>
+                <origin xyz="0 0 0" rpy="0 0 0" />
+                <geometry>
+                    <mesh filename="package://excavator_description/meshes/chassis.STL" />
+                </geometry>
+                <material name="">
+                    <color rgba="0.52941 0.54902 0.54902 1" />
+                </material>
+            </visual>
+            <collision>
+                <origin xyz="0 0 0" rpy="0 0 0" />
+                <geometry>
+                    <mesh filename="package://excavator_description/meshes/chassis.STL" />
                 </geometry>
             </collision>
@@ -184,38 +166,21 @@
         <link name="wheel1">
             <inertial>
-                <origin
-                xyz="0 -0.0095819 7.2858E-17"
-                rpy="0 0 0" />
-                <mass
-                value="0.41779" />
-                <inertia
-                ixx="0.00011232"
-                ixy="1.3277E-20"
-                ixz="2.9754E-21"
-                iyy="0.00019137"
-                iyz="-5.9467E-19"
-                izz="0.00010559" />
-            </inertial>
-            <visual>
-                <origin
-                xyz="0 0 0"
-                rpy="0 0 0" />
-                <geometry>
-                <mesh
-                    filename="package://excavator_description/meshes/wheel1.STL" />
-                </geometry>
-                <material
-                name="">
-                <color
-                    rgba="0.8 0.4 0.4 1" />
-                </material>
-            </visual>
-            <collision>
-                <origin
-                xyz="0 0 0"
-                rpy="0 0 0" />
-                <geometry>
-                <mesh
-                    filename="package://excavator_description/meshes/wheel1.STL" />
+                <origin xyz="0 -0.0095819 7.2858E-17" rpy="0 0 0" />
+                <mass value="0.41779" />
+                <inertia ixx="0.00011232" ixy="1.3277E-20" ixz="2.9754E-21" iyy="0.00019137" iyz="-5.9467E-19" izz="0.00010559" />
+            </inertial>
+            <visual>
+                <origin xyz="0 0 0" rpy="0 0 0" />
+                <geometry>
+                    <mesh filename="package://excavator_description/meshes/wheel1.STL" />
+                </geometry>
+                <material name="">
+                    <color rgba="0.8 0.4 0.4 1" />
+                </material>
+            </visual>
+            <collision>
+                <origin xyz="0 0 0" rpy="0 0 0" />
+                <geometry>
+                    <mesh filename="package://excavator_description/meshes/wheel1.STL" />
                 </geometry>
             </collision>
@@ -223,54 +188,30 @@
         <!-- wheel1_joint -->
         <joint name="wheel1_joint" type="continuous">
-        <origin
-            xyz="0.13707 -0.08 -0.01"
-            rpy="0 0 0" />
-        <parent
-            link="chassis" />
-        <child
-            link="wheel1" />
-        <axis
-            xyz="0 1 0" />
-        <limit
-            effort="100"
-            velocity="6" />
+            <origin xyz="0.13707 -0.08 -0.01" rpy="0 0 0" />
+            <parent link="chassis" />
+            <child link="wheel1" />
+            <axis xyz="0 1 0" />
+            <limit effort="100" velocity="6" />
         </joint>
         <!-- wheel2 -->
         <link name="wheel2">
             <inertial>
-                <origin
-                xyz="0 -0.0095819 7.2858E-17"
-                rpy="0 0 0" />
-                <mass
-                value="0.41779" />
-                <inertia
-                ixx="0.00011232"
-                ixy="1.3277E-20"
-                ixz="2.9754E-21"
-                iyy="0.00019137"
-                iyz="-5.9486E-19"
-                izz="0.00010559" />
-            </inertial>
-            <visual>
-                <origin
-                xyz="0 0 0"
-                rpy="0 0 0" />
-                <geometry>
-                <mesh
-                    filename="package://excavator_description/meshes/wheel2.STL" />
-                </geometry>
-                <material
-                name="carbon_steel">
-                <color
-                    rgba="0.4 0.8 0.4 1" />
-                </material>
-            </visual>
-            <collision>
-                <origin
-                xyz="0 0 0"
-                rpy="0 0 0" />
-                <geometry>
-                <mesh
-                    filename="package://excavator_description/meshes/wheel2.STL" />
+                <origin xyz="0 -0.0095819 7.2858E-17" rpy="0 0 0" />
+                <mass value="0.41779" />
+                <inertia ixx="0.00011232" ixy="1.3277E-20" ixz="2.9754E-21" iyy="0.00019137" iyz="-5.9486E-19" izz="0.00010559" />
+            </inertial>
+            <visual>
+                <origin xyz="0 0 0" rpy="0 0 0" />
+                <geometry>
+                    <mesh filename="package://excavator_description/meshes/wheel2.STL" />
+                </geometry>
+                <material name="carbon_steel">
+                    <color rgba="0.4 0.8 0.4 1" />
+                </material>
+            </visual>
+            <collision>
+                <origin xyz="0 0 0" rpy="0 0 0" />
+                <geometry>
+                    <mesh filename="package://excavator_description/meshes/wheel2.STL" />
                 </geometry>
             </collision>
@@ -278,357 +219,196 @@
         <!-- wheel2_joint -->
         <joint name="wheel2_joint" type="continuous">
-        <origin
-            xyz="-0.12293 -0.08 -0.01"
-            rpy="0 0 0" />
-        <parent
-            link="chassis" />
-        <child
-            link="wheel2" />
-        <axis
-            xyz="0 1 0" />
-        <limit
-            effort="100"
-            velocity="6" />
+            <origin xyz="-0.12293 -0.08 -0.01" rpy="0 0 0" />
+            <parent link="chassis" />
+            <child link="wheel2" />
+            <axis xyz="0 1 0" />
+            <limit effort="100" velocity="6" />
         </joint>
         <!-- wheel3 -->
         <link name="wheel3">
-        <inertial>
-            <origin
-            xyz="0 0.0095819 1.7347E-18"
-            rpy="0 0 0" />
-            <mass
-            value="0.41779" />
-            <inertia
-            ixx="0.00011232"
-            ixy="1.6502E-21"
-            ixz="-7.4622E-22"
-            iyy="0.00019137"
-            iyz="3.3884E-22"
-            izz="0.00010559" />
-        </inertial>
-        <visual>
-            <origin
-            xyz="0 0 0"
-            rpy="0 0 0" />
-            <geometry>
-            <mesh
-                filename="package://excavator_description/meshes/wheel3.STL" />
-            </geometry>
-            <material
-            name="">
-            <color
-                rgba="0.4 0.8 0.4 1" />
-            </material>
-        </visual>
-        <collision>
-            <origin
-            xyz="0 0 0"
-            rpy="0 0 0" />
-            <geometry>
-            <mesh
-                filename="package://excavator_description/meshes/wheel3.STL" />
-            </geometry>
-        </collision>
+            <inertial>
+                <origin xyz="0 0.0095819 1.7347E-18" rpy="0 0 0" />
+                <mass value="0.41779" />
+                <inertia ixx="0.00011232" ixy="1.6502E-21" ixz="-7.4622E-22" iyy="0.00019137" iyz="3.3884E-22" izz="0.00010559" />
+            </inertial>
+            <visual>
+                <origin xyz="0 0 0" rpy="0 0 0" />
+                <geometry>
+                    <mesh filename="package://excavator_description/meshes/wheel3.STL" />
+                </geometry>
+                <material name="">
+                    <color rgba="0.4 0.8 0.4 1" />
+                </material>
+            </visual>
+            <collision>
+                <origin xyz="0 0 0" rpy="0 0 0" />
+                <geometry>
+                    <mesh filename="package://excavator_description/meshes/wheel3.STL" />
+                </geometry>
+            </collision>
         </link>
         <!-- wheel3_joint -->
         <joint name="wheel3_joint" type="continuous">
-        <origin
-            xyz="-0.12293 0.08 -0.01"
-            rpy="0 0 0" />
-        <parent
-            link="chassis" />
-        <child
-            link="wheel3" />
-        <axis
-            xyz="0 1 0" />
-        <limit
-            effort="100"
-            velocity="6" />
+            <origin xyz="-0.12293 0.08 -0.01" rpy="0 0 0" />
+            <parent link="chassis" />
+            <child link="wheel3" />
+            <axis xyz="0 1 0" />
+            <limit effort="100" velocity="6" />
         </joint>
         <!-- wheel4 -->
         <link name="wheel4">
-        <inertial>
-            <origin
-            xyz="0 0.0095819 1.7347E-18"
-            rpy="0 0 0" />
-            <mass
-            value="0.41779" />
-            <inertia
-            ixx="0.00011232"
-            ixy="-3.3874E-22"
-            ixz="-6.774E-22"
-            iyy="0.00019137"
-            iyz="-7.2041E-23"
-            izz="0.00010559" />
-        </inertial>
-        <visual>
-            <origin
-            xyz="0 0 0"
-            rpy="0 0 0" />
-            <geometry>
-            <mesh
-                filename="package://excavator_description/meshes/wheel4.STL" />
-            </geometry>
-            <material
-            name="">
-            <color
-                rgba="0.8 0.4 0.4 1" />
-            </material>
-        </visual>
-        <collision>
-            <origin
-            xyz="0 0 0"
-            rpy="0 0 0" />
-            <geometry>
-            <mesh
-                filename="package://excavator_description/meshes/wheel4.STL" />
-            </geometry>
-        </collision>
+            <inertial>
+                <origin xyz="0 0.0095819 1.7347E-18" rpy="0 0 0" />
+                <mass value="0.41779" />
+                <inertia ixx="0.00011232" ixy="-3.3874E-22" ixz="-6.774E-22" iyy="0.00019137" iyz="-7.2041E-23" izz="0.00010559" />
+            </inertial>
+            <visual>
+                <origin xyz="0 0 0" rpy="0 0 0" />
+                <geometry>
+                    <mesh filename="package://excavator_description/meshes/wheel4.STL" />
+                </geometry>
+                <material name="">
+                    <color rgba="0.8 0.4 0.4 1" />
+                </material>
+            </visual>
+            <collision>
+                <origin xyz="0 0 0" rpy="0 0 0" />
+                <geometry>
+                    <mesh filename="package://excavator_description/meshes/wheel4.STL" />
+                </geometry>
+            </collision>
         </link>
         <!-- wheel4_joint -->
         <joint name="wheel4_joint" type="continuous">
-        <origin
-            xyz="0.13707 0.08 -0.01"
-            rpy="0 0 0" />
-        <parent
-            link="chassis" />
-        <child
-            link="wheel4" />
-        <axis
-            xyz="0 1 0" />
-        <limit
-            effort="100"
-            velocity="6" />
+            <origin xyz="0.13707 0.08 -0.01" rpy="0 0 0" />
+            <parent link="chassis" />
+            <child link="wheel4" />
+            <axis xyz="0 1 0" />
+            <limit effort="100" velocity="6" />
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
Commit message: Fix the Gazebo simulation failing problem(excavator with kinect)

File: src/excavator/excavator_description/urdf/excavator.xacro (robot description, xacro)
@@ -121,4 +121,49 @@
             </plugin>
         </gazebo>
+        <transmission name="trans_table_joint">
+            <type>transmission_interface/SimpleTransmission</type>
+            <joint name="table_joint">
+                <hardwareInterface>hardware_interface/PositionJointInterface</hardwareInterface>
+            </joint>
+            <actuator name="table_joint_motor">
+                <hardwareInterface>hardware_interface/PositionJointInterface</hardwareInterface>
+                <mechanicalReduction>1</mechanicalReduction>
+            </actuator>
+        </transmission>
+        <transmission name="trans_link1_joint">
+            <type>transmission_interface/SimpleTransmission</type>
+            <joint name="link1_joint">
+                <hardwareInterface>hardware_interface/PositionJointInterface</hardwareInterface>
+            </joint>
+            <actuator name="link1_joint_motor">
+                <hardwareInterface>hardware_interface/PositionJointInterface</hardwareInterface>
+                <mechanicalReduction>1</mechanicalReduction>
+            </actuator>
+        </transmission>
+        <transmission name="trans_link2_joint">
+            <type>transmission_interface/SimpleTransmission</type>
+            <joint name="link2_joint">
+                <hardwareInterface>hardware_interface/PositionJointInterface</hardwareInterface>
+            </joint>
+            <actuator name="link2_joint_motor">
+                <hardwareInterface>hardware_interface/PositionJointInterface</hardwareInterface>
+                <mechanicalReduction>1</mechanicalReduction>
+            </actuator>
+        </transmission>
+        <transmission name="trans_ram_joint">
+            <type>transmission_interface/SimpleTransmission</type>
+            <joint name="ram_joint">
+                <hardwareInterface>hardware_interface/PositionJointInterface</hardwareInterface>
+            </joint>
+            <actuator name="ram_joint_motor">
+                <hardwareInterface>hardware_interface/PositionJointInterface</hardwareInterface>
+                <mechanicalReduction>1</mechanicalReduction>
+            </actuator>
+        </transmission>
+        <gazebo>
+            <plugin name="gazebo_ros_control" filename="libgazebo_ros_control.so">
+                <robotNamespace>/</robotNamespace>
+            </plugin>
+        </gazebo>
         <!-- Base Footprint -->
         <link name="base_footprint">

File: src/excavator/excavator_description/urdf/excavator_gazebo.xacro (robot description, xacro)
@@ -4,48 +4,3 @@
     <!-- 调用宏函数 -->
     <xacro:excavator/>
-    <transmission name="trans_table_joint">
-        <type>transmission_interface/SimpleTransmission</type>
-        <joint name="table_joint">
-            <hardwareInterface>hardware_interface/PositionJointInterface</hardwareInterface>
-        </joint>
-        <actuator name="table_joint_motor">
-            <hardwareInterface>hardware_interface/PositionJointInterface</hardwareInterface>
-            <mechanicalReduction>1</mechanicalReduction>
-        </actuator>
-    </transmission>
-    <transmission name="trans_link1_joint">
-        <type>transmission_interface/SimpleTransmission</type>
-        <joint name="link1_joint">
-            <hardwareInterface>hardware_interface/PositionJointInterface</hardwareInterface>
-        </joint>
-        <actuator name="link1_joint_motor">
-            <hardwareInterface>hardware_interface/PositionJointInterface</hardwareInterface>
-            <mechanicalReduction>1</mechanicalReduction>
-        </actuator>
-    </transmission>
-    <transmission name="trans_link2_joint">
-        <type>transmission_interface/SimpleTransmission</type>
-        <joint name="link2_joint">
-            <hardwareInterface>hardware_interface/PositionJointInterface</hardwareInterface>
-        </joint>
-        <actuator name="link2_joint_motor">
-            <hardwareInterface>hardware_interface/PositionJointInterface</hardwareInterface>
-            <mechanicalReduction>1</mechanicalReduction>
-        </actuator>
-    </transmission>
-    <transmission name="trans_ram_joint">
-        <type>transmission_interface/SimpleTransmission</type>
-        <joint name="ram_joint">
-            <hardwareInterface>hardware_interface/PositionJointInterface</hardwareInterface>
-        </joint>
-        <actuator name="ram_joint_motor">
-            <hardwareInterface>hardware_interface/PositionJointInterface</hardwareInterface>
-            <mechanicalReduction>1</mechanicalReduction>
-        </actuator>
-    </transmission>
-    <gazebo>
-        <plugin name="gazebo_ros_control" filename="libgazebo_ros_control.so">
-            <robotNamespace>/</robotNamespace>
-        </plugin>
-    </gazebo>
 </robot>
